File: battery-test-board/battery-test-board.kicad_pcb (KiCad board)
At the start: 2 copper layers, 126.1 x 134.2 mm, 79 parts, among them J1 Conn_02x04_Odd_Even, J10 Screw_Terminal_01x02, J2 Conn_02x04_Odd_Even, J3 Screw_Terminal_01x02, J4 Screw_Terminal_01x02, J5 Screw_Terminal_01x02, J6 Screw_Terminal_01x02, J7 Conn_02x04_Odd_Even, J8 connector, J9 connector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

Commit message: Fixed many little issues
Parts:
- H1, H2, H3, H4, H5, H6, H7, H8: value MountingHole_3.2mm_M3_Pad_Via -> MountingHole_Pad
- R10, R12, R6, R8: value R -> 510k
- TH0, TH1, TH2, TH3: footprint Connector_PinHeader_2.54mm:PinHeader_1x02_P2.54mm_Vertical -> thermister:thermister-solderin
- moved H4 100.3 mm to (150.5, 157.0)
- moved H3 99.9 mm to (31.2, 157.1)
- moved H5 64.5 mm to (64.8, 63.0)
- moved H6 64.5 mm to (115.6, 63.0)
- moved H8 45.4 mm to (115.6, 127.5)
- moved H7 44.4 mm to (64.8, 127.5)
- moved J7 6.41 mm to (144.0, 54.1), turned to 90 degrees
- moved TH1 4.47 mm to (65.2, 92.7), turned to 0 degrees
- moved TH3 4.47 mm to (116.0, 92.7), turned to 0 degrees
- moved TH0 4.47 mm to (39.8, 92.7), turned to 0 degrees
- moved TH2 4.47 mm to (90.6, 92.7), turned to 0 degrees
- moved R16 4.13 mm to (141.0, 54.6), turned to 90 degrees
- moved D10 0.41 mm to (124.0, 28.8)
- moved D8 0.41 mm to (139.7, 28.8)
- moved REF** 0.25 mm to (67.6, 152.1)
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Connections:
- net relay_v renamed relay_s
- TH0 pad 1: Net-(R6-Pad2) -> GND
- TH0 pad 2: GND -> Net-(R6-Pad2)
- TH1 pad 1: Net-(R8-Pad1) -> GND
- TH1 pad 2: GND -> Net-(R8-Pad1)
- TH2 pad 1: Net-(R10-Pad2) -> GND
- TH2 pad 2: GND -> Net-(R10-Pad2)
- TH3 pad 1: Net-(R12-Pad1) -> GND
- TH3 pad 2: GND -> Net-(R12-Pad1)
Routing:
- net relay_s: track 112.8 -> 121.2 mm
- net +12V: track 358.6 -> 365.8 mm
- net Net-(J7-Pad8): track 8.45 -> 14.3 mm
- net Net-(J7-Pad6): track 17.3 -> 19.4 mm
- net Net-(J7-Pad4): track 25.8 -> 23.8 mm
- net Net-(J7-Pad2): track 4.70 -> 3.29 mm
- net Net-(F3-Pad2): track 33.4 -> 34.0 mm
- net Net-(BT2-Pad2): track 97.2 -> 97.8 mm
- net GND: vias 1 -> 0
Other:
- board size 126.1 x 134.2 mm -> 126.1 x 134.7 mm
- board text added: "Battery Tester"
- board text added: "Charge Bank Select"
- board text added: "Connects Li-Ion cells in banks to a battery test system."
- board text added: "Sense Bank Select"
- board text added: "Sense Selected"
- board text added: "Termination Select: Jump each row on on only one board"
- board text added: "Use both Bank Selects select which bank this board is. Select the same value on both. Do not select the same bank on multiple boards."
- board text added: "V1.0 2022/03/30"
- board text removed: "Bank Select A"
- board text removed: "Bank Select B"
- board text removed: "Battery Tester V1.0 2022/03/30"
- board text removed: "Jump each row on J7 on only one board"
- board text removed: "Measure Selected"
- board text removed: "Use Bank Select A&B to select which bank this board is. Select the same value on both. Do not select the same bank on multiple boards."
