File: battery-test-board/battery-test-board.kicad_pcb (KiCad board)
At the start: 2 copper layers, 126.1 x 134.7 mm, 79 parts, among them J1 Conn_02x04_Odd_Even, J10 Screw_Terminal_01x02, J2 Conn_02x04_Odd_Even, J3 Screw_Terminal_01x02, J4 Screw_Terminal_01x02, J5 Screw_Terminal_01x02, J6 Screw_Terminal_01x02, J7 Conn_02x04_Odd_Even, J8 connector, J9 connector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

Commit message: Fixed a few issues missed last time
Parts:
- added REF**: github-oresat-battery-testing-qr, oresat-logo:github-oresat-battery-testing-qr, F.Cu at (115.1, 154.4)
- moved U7 0.13 mm to (117.0, 140.3)
- moved H4 0.13 mm to (150.5, 157.1)
- moved U4 0.13 mm to (65.4, 137.8)
Routing:
- net GND: vias 0 -> 53
Other:
- outline, holes or cut-outs redrawn
- board text added: "12V 200mA Relay Power"
- board text added: "More info: github.com/oresat/ oresat-battery-testing"
- board text removed: "J10 12V 200mA Relay Power"
