File: battery-test-board/battery-test-board.kicad_sch (KiCad schematic)
At the start: 58 parts, among them J1 Conn_02x04_Odd_Even, J10 Screw_Terminal_01x02, J2 Conn_02x04_Odd_Even, J3 Screw_Terminal_01x02, J4 Screw_Terminal_01x02, J5 Screw_Terminal_01x02, J6 Screw_Terminal_01x02, J7 Conn_02x04_Odd_Even, J8 Conn_02x20_Odd_Even, J9 Conn_02x20_Odd_Even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

Commit message: Updated footprints and PCB
Parts:
- added D1, D10, D2, D4, D5, D7, D8, D9: diode, Diode_SMD:D_0805_2012Metric, symbol Device:D
- added D15, D16: Green, LED_SMD:LED_1206_3216Metric, symbol Device:LED
- added R17: 4k7, Resistor_SMD:R_1206_3216Metric, symbol Device:R
- added R18: 10k, Resistor_SMD:R_1206_3216Metric, symbol Device:R
- BT0, BT1, BT2, BT3: value BK-18650-PC2 -> battery; DPN (none) -> 1; Descrip (none) -> 1; MPN (none) -> BK-18650-PC2
- C1, C2: value C -> 10u
- D11: renamed from D4; value NSR05T40P2T5G -> diode; footprint (none) -> Diode_SMD:D_0805_2012Metric; MPN (none) -> NSR05T40P2T5G
- D12: renamed from D5; value NSR05T40P2T5G -> diode; footprint (none) -> Diode_SMD:D_0805_2012Metric; MPN (none) -> NSR05T40P2T5G
- D13: renamed from D1; value LED -> Amber
- D14: renamed from D2; value LED -> Amber
- D3, D6: value NSR05T40P2T5G -> diode; footprint (none) -> Diode_SMD:D_0805_2012Metric; MPN (none) -> NSR05T40P2T5G
- J8, J9: value Conn_02x20_Odd_Even -> (none); footprint Connector_PinSocket_2.54mm:PinSocket_2x20_P2.54mm_Vertical -> (none); MPN (none) -> 732-5401-ND
- Q1, Q2: value PJA3412-AU_R1_000A1 -> mosfet; MPN (none) -> PJA3412-AU_R1_000A1
- R1, R3: value 330 -> 4k7
- R11, R5, R7, R9: value 1k -> 470
- TH0, TH1, TH2, TH3: DPN (none) -> 490-14854-ND; Descrip (none) -> NTC Thermistor 10k Bead; MPN (none) -> NXFT15XH103FA2B040
- U1, U10, U2, U3, U4, U5, U6, U7, U8, U9: value J104D2C12VDC.15S‎ -> relay; MPN (none) -> J104D2C12VDC.15S‎
Connections:
- net +12V: now also D1.1 (K), D10.1 (K), D16.2 (A), D2.1 (K), D4.1 (K), D5.1 (K), D7.1 (K), D8.1 (K), D9.1 (K)
- net +5V: now also D15.2 (A)
- net GND: now also R17.2, R18.2
- net bank_0c: now also J8.30 (Pin_30), J9.30 (Pin_30); no longer J8.29 (Pin_29), J9.29 (Pin_29)
- net bank_0m: now also J8.29 (Pin_29), J9.29 (Pin_29); no longer J8.30 (Pin_30), J9.30 (Pin_30)
- net bank_1c: now also J8.32 (Pin_32), J9.32 (Pin_32); no longer J8.31 (Pin_31), J9.31 (Pin_31)
- net bank_1m: now also J8.31 (Pin_31), J9.31 (Pin_31); no longer J8.32 (Pin_32), J9.32 (Pin_32)
- net bank_2c: now also J8.34 (Pin_34), J9.34 (Pin_34); no longer J8.33 (Pin_33), J9.33 (Pin_33)
- net bank_2m: now also J8.33 (Pin_33), J9.33 (Pin_33); no longer J8.34 (Pin_34), J9.34 (Pin_34)
- net bank_3c: now also J8.36 (Pin_36), J9.36 (Pin_36); no longer J8.35 (Pin_35), J9.35 (Pin_35)
- net bank_3m: now also J8.35 (Pin_35), J9.35 (Pin_35); no longer J8.36 (Pin_36), J9.36 (Pin_36)
- net batt_0+: now also J8.4 (Pin_4), J9.4 (Pin_4); no longer J8.3 (Pin_3), J9.3 (Pin_3)
- net batt_0-: now also J8.3 (Pin_3), J9.3 (Pin_3); no longer J8.4 (Pin_4), J9.4 (Pin_4)
- net batt_0t: now also J8.20 (Pin_20), J9.20 (Pin_20); no longer J8.19 (Pin_19), J9.19 (Pin_19)
- net batt_1+: now also J8.8 (Pin_8), J9.8 (Pin_8); no longer J8.7 (Pin_7), J9.7 (Pin_7)
- net batt_1-: now also J8.7 (Pin_7), J9.7 (Pin_7); no longer J8.8 (Pin_8), J9.8 (Pin_8)
- net batt_1t: now also J8.19 (Pin_19), J9.19 (Pin_19); no longer J8.20 (Pin_20), J9.20 (Pin_20)
- net batt_2+: now also J8.12 (Pin_12), J9.12 (Pin_12); no longer J8.11 (Pin_11), J9.11 (Pin_11)
- net batt_2-: now also J8.11 (Pin_11), J9.11 (Pin_11); no longer J8.12 (Pin_12), J9.12 (Pin_12)
- net batt_2t: now also J8.24 (Pin_24), J9.24 (Pin_24); no longer J8.23 (Pin_23), J9.23 (Pin_23)
- net batt_3+: now also J8.16 (Pin_16), J9.16 (Pin_16); no longer J8.15 (Pin_15), J9.15 (Pin_15)
- net batt_3-: now also J8.15 (Pin_15), J9.15 (Pin_15); no longer J8.16 (Pin_16), J9.16 (Pin_16)
- net batt_3t: now also J8.23 (Pin_23), J9.23 (Pin_23); no longer J8.24 (Pin_24), J9.24 (Pin_24)
- net relay_c: now also D2.2 (A), D4.2 (A), D7.2 (A), D9.2 (A); no longer D3.2 (A)
- net relay_v: now also D3.2 (A), D1.2 (A), D10.2 (A), D5.2 (A), D8.2 (A)
- new net: D15.1 (K), R17.1
- new net: D16.1 (K), R18.1
Other:
- note added: "+5v from labjack for thermisters"
- note added: "12v@200mA"
- note added: "According to LabJack guidelines, needs 1M resistors on one input even though they are differential"
- note added: "Jump all positions on only 1 board"
- note added: "Jump one position on J1 and J2 to select which bank this board is"
- note added: "Power Status"
- note added: "Power supply connectors"
- note added: "batt_X+ : Battery + voltage measurement batt_X- : Battery - voltage measurement batt_Xt : Battery temperature measurement bank_Yc : Bank Y charge select bank_Ym : Bank Y measurement select"
- note added: "charge_X+ : Charger X + input charge_X- : Charger X - input"
- note added: "jumpers (pick 1)"
- note added: "relay_c : Charge control relay power"
- note added: "relay_v : Voltage / temperature relay power"
- moved on the sheet: BT0, BT1, BT2, BT3, D11, F1, F2, F3, F4, J10, J3, J4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

Commit message: Fixed silk screen and a few other things
Parts:
- J8, J9: value (none) -> connector; footprint (none) -> Connector_IDC:IDC-Header_2x20_P2.54mm_Vertical
Connections:
- net GND: now also D14.1 (K); no longer R3.1
- net at R3.2: now also D14.2 (A); no longer D14.1 (K)
- net at J2.1 (Pin_1), J2.3 (Pin_3), J2.5 (Pin_5)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: now also R3.1; no longer D14.2 (A)
Other:
- moved on the sheet: D14, R3

Commit message: Finished BOM
Parts:
- BT0, BT1, BT2, BT3: value battery -> (none); footprint Battery:BatteryHolder_MPD_BH-18650-PC2 -> (none); DPN 1 -> BK-18650-PC2-ND; Descrip 1 -> Battery Holder (Open) 18650 1 Cell PC Pin
- C1, C2: value 10u -> (none); footprint Capacitor_SMD:C_1206_3216Metric -> (none); DPN (none) -> 1276-1075-1-ND; Descrip (none) -> 10 µF ±10% 25V Ceramic Capacitor X5R 1206 (3216 Metric); MPN (none) -> CL31A106KAHNNNE
- D1, D10, D11, D12, D2, D3, D4, D5, D6, D7, D8, D9: value diode -> (none); footprint Diode_SMD:D_0805_2012Metric -> (none); DPN (none) -> NSR05T40P2T5GOSCT-ND; Descrip (none) -> Diode Schottky 40 V 500mA (DC) Surface Mount SOD-923
- D13, D14: value Amber -> (none); footprint LED_SMD:LED_1206_3216Metric -> (none); DPN (none) -> 732-4988-1-ND; Descrip (none) -> Amber 605nm LED Indication - Discrete 2V 1206 (3216 Metric); MPN (none) -> 150120AS75000
- D15, D16: value Green -> (none); footprint LED_SMD:LED_1206_3216Metric -> (none); DPN (none) -> 732-4993-1-ND; Descrip (none) -> Green 570nm LED Indication - Discrete 2V 1206 (3216 Metric); MPN (none) -> 150120VS75000
- F1, F2, F3, F4: value Polyfuse 2A -> (none); footprint Fuse:Fuse_0805_2012Metric -> (none); DPN (none) -> F2868CT-ND; Descrip (none) -> Polymeric PTC Resettable Fuse 33V 1.1 A Ih Surface Mount 29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; MPN (none) -> 2920L100PR
- J1, J2, J7: value Conn_02x04_Odd_Even -> (none); footprint Connector_PinSocket_2.54mm:PinSocket_2x04_P2.54mm_Vertical -> (none); DPN (none) -> 1849-PR20204VBDN-ND; Descrip (none) -> Connector Header Through Hole 8 position 0.100" (2.54mm); MPN (none) -> PR20204VBDN
- J10, J3, J4, J5, J6: value Screw_Terminal_01x02 -> (none); footprint TerminalBlock:TerminalBlock_Altech_AK300-2_P5.00mm -> (none); DPN (none) -> 2057-EBAA-02-C-ND; Descrip (none) -> 2 Position Wire to Board Terminal Block Horizontal with Boa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; MPN (none) -> EBAA-02-C
- J8, J9: value connector -> (none); footprint Connector_IDC:IDC-Header_2x20_P2.54mm_Vertical -> (none); DPN (none) -> 732-5401-ND; Descrip (none) -> Connector Header Through Hole 40 position 0.100" (2.54mm)
- Q1, Q2: value mosfet -> (none); footprint Package_TO_SOT_SMD:SOT-23 -> (none); DPN (none) -> 3757-PJA3412-AU_R1_000A1CT-ND; Descrip (none) -> N-Channel 20 V 4.1A (Ta) 1.25W (Ta) Surface Mount SOT-23k
- R1, R17, R3: value 4k7 -> (none); footprint Resistor_SMD:R_1206_3216Metric -> (none); DPN (none) -> RMCF1206FT4K70CT-ND; Descrip (none) -> 4.7 kOhms ±1% 0.25W, 1/4W Chip Resistor 1206 (3216 Metric) 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; MPN (none) -> RMCF1206FT4K70
- R10, R12, R6, R8: value R -> (none); footprint Resistor_SMD:R_1206_3216Metric -> (none); DPN (none) -> RMCF1206FT510KCT-ND; Descrip (none) -> 510 kOhms ±1% 0.25W, 1/4W Chip Resistor 1206 (3216 Metric) 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; MPN (none) -> RMCF1206FT510K
- R11, R5, R7, R9: value 470 -> (none); footprint Resistor_SMD:R_1206_3216Metric -> (none); DPN (none) -> RMCF1206FT470RCT-ND; Descrip (none) -> 470 Ohms ±1% 0.25W, 1/4W Chip Resistor 1206 (3216 Metric) A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; MPN (none) -> RMCF1206FT470R
- R13, R14, R15, R16: value 1M -> (none); footprint Resistor_SMD:R_1206_3216Metric -> (none); DPN (none) -> RMCF1206FT1M00CT-ND; Descrip (none) -> 1 MOhms ±1% 0.25W, 1/4W Chip Resistor 1206 (3216 Metric) Au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; MPN (none) -> RMCF1206FT1M00
- R18: value 10k -> (none); footprint Resistor_SMD:R_1206_3216Metric -> (none); DPN (none) -> RMCF1206FT10K0CT-ND; Descrip (none) -> 10 kOhms ±1% 0.25W, 1/4W Chip Resistor 1206 (3216 Metric) A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; MPN (none) -> RMCF1206FT10K0
- R2, R4: value 10K -> (none); footprint Resistor_SMD:R_1206_3216Metric -> (none); DPN (none) -> RMCF1206FT10K0CT-ND; Descrip (none) -> 10 kOhms ±1% 0.25W, 1/4W Chip Resistor 1206 (3216 Metric) A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; MPN (none) -> RMCF1206FT10K0
- TH0, TH1, TH2, TH3: value Thermistor -> (none); footprint Connector_PinHeader_2.54mm:PinHeader_1x02_P2.54mm_Vertical -> (none); DPN 490-14854-ND -> 490-12817-ND; MPN NXFT15XH103FA2B040 -> NXFT15XH103FA1B025
- U1, U10, U2, U3, U4, U5, U6, U7, U8, U9: value relay -> (none); footprint relay:relay-dpdt-.3in -> (none); DPN (none) -> 2449-J104D2C12VDC.15S-ND; Descrip (none) -> General Purpose Relay DPDT
Connections:
- net charge_2+: now also U7.13 (c3); no longer U7.4 (c1)
- net charge_2-: now also U7.4 (c1); no longer U7.13 (c3)
- net at BT2.2 (-), U6.9 (no2): now also U7.8 (no1); no longer U7.9 (no2)
- net at F3.2: now also U7.9 (no2); no longer U7.8 (no1)
Other:
- moved on the sheet: D7

Commit message: Fixed many little issues
Parts:
- added H1, H2, H3, H4, H5, H6, H7, H8: MountingHole_Pad, MountingHole:MountingHole_3.2mm_M3_Pad_Via, symbol Mechanical:MountingHole_Pad
- BT0, BT1, BT2, BT3: value (none) -> battery; footprint (none) -> Battery:BatteryHolder_MPD_BH-18650-PC2
- C1, C2: value (none) -> 10u; footprint (none) -> Capacitor_SMD:C_1206_3216Metric
- D1, D10, D11, D12, D2, D3, D4, D5, D6, D7, D8, D9: value (none) -> diode; footprint (none) -> Diode_SMD:D_0805_2012Metric
- D13, D14: value (none) -> Amber; footprint (none) -> LED_SMD:LED_1206_3216Metric
- D16: value (none) -> Green; footprint (none) -> LED_SMD:LED_1206_3216Metric
- F1, F2, F3, F4: value (none) -> Polyfuse 2A; footprint (none) -> Fuse:Fuse_2920_7451Metric
- J1, J2, J7: value (none) -> Conn_02x04_Odd_Even; footprint (none) -> Connector_PinSocket_2.54mm:PinSocket_2x04_P2.54mm_Vertical
- J10, J3, J4, J5, J6: value (none) -> Screw_Terminal_01x02; footprint (none) -> TerminalBlock:TerminalBlock_Altech_AK300-2_P5.00mm
- J8, J9: value (none) -> connector; footprint (none) -> Connector_IDC:IDC-Header_2x20_P2.54mm_Vertical
- Q1, Q2: value (none) -> mosfet; footprint (none) -> Package_TO_SOT_SMD:SOT-23
- R1: symbol Device:R -> Device:R_US
- R10, R12, R6, R8: value (none) -> 510k; footprint (none) -> Resistor_SMD:R_1206_3216Metric; symbol Device:R -> Device:R_US
- R11, R5, R7, R9: value (none) -> 470; footprint (none) -> Resistor_SMD:R_1206_3216Metric; symbol Device:R -> Device:R_US
- R13, R14, R15, R16: value (none) -> 1M; footprint (none) -> Resistor_SMD:R_1206_3216Metric; symbol Device:R -> Device:R_US
- R17, R3: value (none) -> 4k7; footprint (none) -> Resistor_SMD:R_1206_3216Metric; symbol Device:R -> Device:R_US
- R18, R2, R4: value (none) -> 10K; footprint (none) -> Resistor_SMD:R_1206_3216Metric; symbol Device:R -> Device:R_US
- TH0, TH1, TH2, TH3: value (none) -> Thermistor; footprint (none) -> thermister:thermister-solderin
- U1, U10, U2, U3, U4, U5, U6, U7, U8, U9: value (none) -> relay; footprint (none) -> relay:relay-dpdt-.3in
Connections:
- net GND: now also TH0.1, TH1.1, TH2.1, TH3.1, H1.1, H2.1, H3.1, H4.1, H5.1, H6.1, H7.1, H8.1; no longer TH0.2, TH1.2, TH2.2, TH3.2
- net at R10.2, U10.8 (1.no): now also TH2.2; no longer TH2.1
- net at R12.1, U10.9 (2.no): now also TH3.2; no longer TH3.1
- net at R6.2, U5.8 (1.no): now also TH0.2; no longer TH0.1
- net at R8.1, U5.9 (2.no): now also TH1.2; no longer TH1.1
- net relay_v renamed relay_s
- no-connect marks 0 -> 20
Other:
- note added: "+5v from labjack for thermistors"
- note added: "Mounting Holes"
- note added: "relay_s : Voltage / temperature relay power"
- note removed: "+5v from labjack for thermisters"
- note removed: "relay_v : Voltage / temperature relay power"
- moved on the sheet: TH0, TH1, TH2, TH3

Commit message: Fixed a few issues missed last time
Parts:
- BT0, BT1, BT2, BT3: value battery -> (none); footprint Battery:BatteryHolder_MPD_BH-18650-PC2 -> (none)
- C1, C2: value 10u -> (none); footprint Capacitor_SMD:C_1206_3216Metric -> (none)
- D1, D10, D11, D12, D2, D3, D4, D5, D6, D7, D8, D9: value diode -> (none); footprint Diode_SMD:D_0805_2012Metric -> (none)
- D13, D14: value Amber -> (none); footprint LED_SMD:LED_1206_3216Metric -> (none)
- D16: value Green -> (none); footprint LED_SMD:LED_1206_3216Metric -> (none)
- F1, F2, F3, F4: value Polyfuse 2A -> (none); footprint Fuse:Fuse_2920_7451Metric -> (none)
- H1, H2, H3, H4, H5, H6, H7, H8: value MountingHole_Pad -> (none); footprint MountingHole:MountingHole_3.2mm_M3_Pad_Via -> (none)
- J1, J2, J7: value Conn_02x04_Odd_Even -> (none); footprint Connector_PinSocket_2.54mm:PinSocket_2x04_P2.54mm_Vertical -> (none)
- J10, J3, J4, J5, J6: value Screw_Terminal_01x02 -> (none); footprint TerminalBlock:TerminalBlock_Altech_AK300-2_P5.00mm -> (none)
- J8, J9: value connector -> (none); footprint Connector_IDC:IDC-Header_2x20_P2.54mm_Vertical -> (none)
- Q1, Q2: value mosfet -> (none); footprint Package_TO_SOT_SMD:SOT-23 -> (none)
- R10, R12, R6, R8: value 510k -> (none); footprint Resistor_SMD:R_1206_3216Metric -> (none)
- R11, R5, R7, R9: value 470 -> (none); footprint Resistor_SMD:R_1206_3216Metric -> (none)
- R13, R14, R15, R16: value 1M -> (none); footprint Resistor_SMD:R_1206_3216Metric -> (none)
- R17, R3: value 4k7 -> (none); footprint Resistor_SMD:R_1206_3216Metric -> (none)
- R18, R2, R4: value 10K -> (none); footprint Resistor_SMD:R_1206_3216Metric -> (none)
- TH0, TH1, TH2, TH3: value Thermistor -> (none); footprint thermister:thermister-solderin -> (none)
- U1, U10, U2, U3, U4, U5, U6, U7, U8, U9: value relay -> (none); footprint relay:relay-dpdt-.3in -> (none)
