File: labjack-connector/labjack-connector.kicad_sch (KiCad schematic)
At the start: 2 parts, among them J1 connector, J2 DB37_Male

Commit message: Added part number
Parts:
- J2: DPN (none) -> AE10986-ND; Descrip (none) -> CONN D-SUB PLUG 37POS R/A SLDR; MPN (none) -> A-DS 37 A/KG-T2S; Manufacturer (none) -> Assmann WSW Components
Changed lines of the file:
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@@
+      (effects (font (size 1.27 1.27)) hide)
+    )
+    (property "DPN" "AE10986-ND" (id 4) (at 83.82 77.47 0)
+      (effects (font (size 1.27 1.27)) hide)
+    )
+    (property "Descrip" "CONN D-SUB PLUG 37POS R/A SLDR" (id 5) (at 83.82 77.47 0)
+      (effects (font (size 1.27 1.27)) hide)
+    )
+    (property "MPN" "A-DS 37 A/KG-T2S" (id 6) (at 83.82 77.47 0)
+      (effects (font (size 1.27 1.27)) hide)
+    )
+    (property "Manufacturer" "Assmann WSW Components" (id 7) (at 83.82 77.47 0)
       (effects (font (size 1.27 1.27)) hide)
     )
